File: board_0.0.1/Board_v0.0..1/FandI.kicad_sch (KiCad schematic)
At the start: 10 parts, among them U3 TC4424A

Commit message: iginition & fuel
Parts:
- added D10, D5, D6, D9: D, Diode_THT:D_DO-35_SOD27_P7.62mm_Horizontal, symbol Device:D
- added D3, D4, D7, D8: LED, LED_THT:LED_D3.0mm, symbol Device:LED
- added Q1, Q2, Q3, Q4: Q_NMOS_GDS, Package_TO_SOT_THT:TO-220-3_Horizontal_TabDown, symbol Device:Q_NMOS_GDS
- added R15, R16, R21, R22: 100k, Resistor_THT:R_Axial_DIN0204_L3.6mm_D1.6mm_P5.08mm_Horizontal, symbol Device:R
- added R17, R18, R23, R24: 1k, Resistor_THT:R_Axial_DIN0204_L3.6mm_D1.6mm_P5.08mm_Horizontal, symbol Device:R
- added R19, R20, R25, R26: 2.4k, Resistor_THT:R_Axial_DIN0204_L3.6mm_D1.6mm_P5.08mm_Horizontal, symbol Device:R
Connections:
- net GND: now also Q1.3 (S), Q2.3 (S), Q3.3 (S), Q4.3 (S), R15.2, R16.1, R21.2, R22.1
- new net: D10.2 (A), D8.1 (K)
- new net: D8.2 (A), R26.1
- new net: Q3.1 (G), R23.1
- new net: D7.1 (K), D9.2 (A)
- new net: Q4.1 (G), R24.1
- new net: D4.1 (K), D6.2 (A)
- new net: D4.2 (A), R20.1
- new net: D7.2 (A), R25.1
- new net: Q1.1 (G), R17.1
- new net: Q2.1 (G), R18.1
- new net: D3.1 (K), D5.2 (A)
- new net: D3.2 (A), R19.1
- new net 12V-SW: R19.2, R20.2, R25.2, R26.2
- new net INJ-1-OUT: D5.1 (K), Q1.2 (D)
- new net INJ-2-OUT: D9.1 (K), Q3.2 (D)
- new net INJ-3-OUT: D10.1 (K), Q4.2 (D)
- new net INJ-4-OUT: D6.1 (K), Q2.2 (D)
- new net MCU-D10: R22.2, R24.2
- new net MCU-D11: R16.2, R18.2
- new net MCU-D8: R15.1, R17.2
- new net MCU-D9: R21.1, R23.2
Other:
- note added: "Injector Driver 1"
- note added: "Injector Driver 2"
- note added: "Injector Driver 3"
- note added: "Injector Driver 4"
